File: DC_DC.kicad_sch (KiCad schematic)
At the start: 22 parts

Commit message: schematic work
Parts:
- C4: renamed from C?; value C_Small -> 100n
- R1: renamed from R?; value R_Small -> 20k
- U1: renamed from U?; LCSC (none) -> C347460
- gave numbers to parts that had none: 19
Connections:
- net GND1 renamed GND
- net GND: no longer D2.1 (K)
Other:
- note added: "R8 Current limiting, dampens parasitic osc. R9 Bleeder / sets state during power up"
- note added: "VREF provides charging current RC is an oscillator programmed by connecting resistor RT (R6?) to VREF and capacitor CT to ground"
- moved on the sheet: C1, C7, D1, D2, L1, R10, R2, R4, R5, R6, R9
